File: H401/KiCAD/Test1.kicad_sch (KiCad schematic)
At the start: 65 parts, among them J1 Conn_Coaxial_Small, P1 USB_C_Plug, Q1 Q_PNP_BCE, SW1 Reset Switch, U1 CH340N, U2 ESP32-PICO-D4, U4 DS1302Z+, U5 AT25SF081-SSHD-X, U6 MI6118, X1 Crystal, X3 Crystal

Commit message: more mods
Connections:
- net at BT1.1 (+), D19.1 (K), U4.5 (CE): now also U2.42 (IO21)
Changed lines of the file:
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@@
+	)
+	(junction
+		(at 224.79 -25.4)
+		(diameter 0)
+		(color 0 0 0 0)
 	)
 	(junction
@@
 	(wire
 		(pts
+			(xy 224.79 -6.35) (xy 224.79 30.48)
+		)
+		(stroke
+			(width 0)
+			(type default)
+		)
+	)
+	(wire
+		(pts
 			(xy 19.05 -8.89) (xy 19.05 20.32)
 		)
@@
 	(wire
 		(pts
-			(xy 314.96 26.67) (xy 314.96 118.11)
-		)
-		(stroke
-			(width 0)
-			(type default)
-		)
-	)
-	(wire
-		(pts
 			(xy 87.63 -24.13) (xy 90.17 -24.13)
 		)
@@
 	(wire
 		(pts
+			(xy 218.44 -25.4) (xy 224.79 -25.4)
+		)
+		(stroke
+			(width 0)
+			(type default)
+		)
+	)
+	(wire
+		(pts
 			(xy 175.26 87.63) (xy 195.58 87.63)
 		)
@@
 	(wire
 		(pts
+			(xy 224.79 -6.35) (xy 218.44 -6.35)
+		)
+		(stroke
+			(width 0)
+			(type default)
+		)
+	)
+	(wire
+		(pts
 			(xy 251.46 -25.4) (xy 261.62 -25.4)
 		)
@@
 	(wire
 		(pts
-			(xy 224.79 26.67) (xy 314.96 26.67)
-		)
-		(stroke
-			(width 0)
-			(type default)
-		)
-	)
-	(wire
-		(pts
 			(xy 41.91 -11.43) (xy 45.72 -11.43)
 		)
@@
 	(wire
 		(pts
-			(xy 224.79 30.48) (xy 224.79 26.67)
-		)
-		(stroke
-			(width 0)
-			(type default)
-		)
-	)
-	(wire
-		(pts
 			(xy 107.95 -22.86) (xy 100.33 -22.86)
 		)
@@
 	(wire
 		(pts
-			(xy 289.56 118.11) (xy 314.96 118.11)
-		)
-		(stroke
-			(width 0)
-			(type default)
-		)
-	)
-	(wire
-		(pts
 			(xy 41.91 -16.51) (xy 35.56 -16.51)
 		)
@@
 		)
 		(stroke
+			(width 0)
+			(type default)
+		)
+	)
+	(wire
+		(pts
+			(xy 218.44 -6.35) (xy 218.44 -25.4)
+		)
+		(stroke
